File: Hardware/uart2pwm/uart2pwm.kicad_pcb (KiCad board)
At the start: 2 copper layers, 63 parts, among them IC1 ATTINY2313A-S, P1 CONN_01X04, P10 LED_G_AN, P11 CONN_01X03, P12 FAN0, P13 CAT, P14 CAT, P15 LED_B_AN, P16 LED_B_AN, P17 FAN1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

Commit message: Finalized first hardware revision
Parts:
- C1, C2, C7, C8: footprint Discret:C1V5 -> Capacitors_SMD:C_0805; moved to B.Cu
- C6: footprint Capacitors_Elko_ThroughHole:Elko_vert_20x10mm_RM5 -> Capacitors_Elko_ThroughHole:Elko_vert_11.5x8mm_RM3.5
- moved Q6 81.3 mm to (61.6, 59.1), turned to 270 degrees
- moved Q3 73.2 mm to (61.6, 62.9), turned to 270 degrees
- moved P17 70.6 mm to (76.7, 63.3)
- moved P12 70.6 mm to (67.8, 63.3)
- moved P11 41.4 mm to (47.0, 49.5)
- moved P2 31.9 mm to (38.7, 28.6), turned to 270 degrees
- moved C4 28.4 mm to (43.8, 45.7)
- moved P15 28.2 mm to (81.2, 55.1)
- moved R18 28.2 mm to (76.1, 57.6)
- moved R20 28.2 mm to (76.1, 55.7)
- moved R22 28.2 mm to (76.1, 51.9)
- moved R24 28.2 mm to (76.1, 53.8)
- moved P9 28.0 mm to (81.2, 42.4)
- moved R10 28.0 mm to (76.1, 44.9)
- moved R12 28.0 mm to (76.1, 43.0)
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Routing:
- net +5V: track 58.3 -> 234.9 mm, vias 0 -> 6
- net +12V: track 8.13 -> 93.9 mm
- net /PWM6_MISO: track 0.00 -> 81.2 mm
- net /PWM7_SCK: track 7.80 -> 82.4 mm
- net /PWM2: track 0.00 -> 57.4 mm
- net /PWM1: track 0.00 -> 44.4 mm
- net GND: track 0.00 -> 43.1 mm, vias 0 -> 6
- net /PWM5_MOSI: track 4.23 -> 46.6 mm
- net /PWM0: track 0.00 -> 34.3 mm
- net /RESET_N: track 0.00 -> 31.1 mm, vias 0 -> 2
- net /RXD_TTL: track 0.00 -> 28.9 mm
- net /TXD_TTL: track 0.00 -> 24.8 mm
- net /PWM4: track 0.00 -> 23.3 mm
- net Net-(Q8-PadD): track 0.00 -> 20.7 mm
- net /PWM3: track 0.00 -> 15.6 mm
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- added copper zone on B.Cu, net GND
Other:
- board outline added: 68 x 46 mm
